Commit message: FIXED OFFSET uvc2308trial_description package

File: autoz_one/src/autozuvc_urdf/urdf/autozuvc_urdf (copy).urdf (robot description, URDF)
Before this commit: robot autozuvc_urdf, 6 links, 5 joints
Joints:
- joint ccontinuous: origin xyz=-0.005 0.355 -0.22 rpy=1.25842195269479 0 0 -> xyz=-0.355 -0.005 -0.22 rpy=1.5708 0 1.5708
- joint cfixed: origin xyz=-0.05 -0.385 0.57 rpy=1.5707963267949 0 0 -> xyz=0.385 -0.05 0.57 rpy=1.5708 0 1.5708
- joint lcontinuous: origin xyz=-0.31 -0.145 -0.12 rpy=2.63245317306069 0 3.14159265358979 -> xyz=0.145 -0.31 -0.12 rpy=-1.5708 0 -1.5708
- joint lfixed: origin xyz=0.00391941090707163 -0.4225 0.2345 rpy=1.5707963267949 0 0 -> xyz=0.4225 0.00391941090707163 0.2345 rpy=1.5708 0 1.5708
- joint rcontinuous: origin xyz=0.31 -0.145 -0.12 rpy=1.65762925454521 0 0 -> xyz=0.145 0.31 -0.12 rpy=1.5708 0 1.5708

File: autoz_one/src/uvcfusion_description/urdf/uvcfusion.xacro (robot description, xacro)
@@ -17,4 +17,6 @@
 <odometryFrame>odom</odometryFrame>
 <robotBaseFrame>base_link</robotBaseFrame>
+<publishWheelTF>true</publishWheelTF>
+<publishWheelJointState>true</publishWheelJointState>
 </plugin>
 </gazebo>
