Commit message: FIXED BLACK RENDERING OF BOT IN RVIZ

File: autoz_one/src/uvc2308trial_description/urdf/materials.xacro (robot description, xacro)
@@ -2,5 +2,5 @@
 <robot name="uvc2308trial" xmlns:xacro="http://www.ros.org/wiki/xacro" >
 <material name="silver">
-  <color rgba="0.700 0.700 0.700 1.000"/>
+  <color rgba="0.7 0.7 0.7 1"/>
 </material>
 </robot>

File: autoz_one/src/uvc2308trial_description/urdf/uvc2308trial.xacro (robot description, xacro)
@@ -2,5 +2,5 @@
 <robot name="uvc2308trial" xmlns:xacro="http://www.ros.org/wiki/xacro">
 <xacro:include filename="$(find uvc2308trial_description)/urdf/materials.xacro" />
-<xacro:include filename="$(find uvc2308trial_description)/urdf/uvc2308trial.trans" />
+<!-- <xacro:include filename="$(find uvc2308trial_description)/urdf/uvc2308trial.trans" /> -->
 <xacro:include filename="$(find uvc2308trial_description)/urdf/uvc2308trial.gazebo" />
 <gazebo>
@@ -13,5 +13,5 @@
 <wheelSeparation>0.64</wheelSeparation>
 <wheelDiameter>0.3</wheelDiameter>
-<torque>0.1</torque>
+<torque>0.2</torque>
 <commandTopic>offset_cmd_vel</commandTopic>
 <odometryTopic>odom</odometryTopic>
@@ -25,5 +25,5 @@
   <inertial>
     <origin rpy="0 0 0" xyz="0.033782226346891105 2.3715430983439135e-06 0.2804808377593937"/>
-    <mass value="10.500150700507"/>
+    <mass value="50.500150700507"/>
     <inertia ixx="51.398406" ixy="0.00093" ixz="-1.652129" iyy="70.361269" iyz="0.000558" izz="79.459893"/>
   </inertial>
